File: eagle/AD8403_SVF/AD8403_SVF_Level.sch (EAGLE design)
At the start: 30 parts, among them IC1 AD8403-DIP24, IC2 NJM2732, IC3 NJM2732

Commit message: Update: eagle files
Parts:
- removed JP7: VGND, pinhead:PINHD-1X2
- removed LED1, LED2: red, led:LED3MM
- removed R4: 100k, rcl:R-EU_0207/7
- removed R7, R8: 220, rcl:R-EU_0207/7
- C1, C2: device rcl:C-EU050-025X075 -> rcl:C-EU025-025X050
- C7: value 0.1uF -> (none)
- IC1: value AD8403-DIP24 -> AD8403-DIP28; device mylib2:AD8403-DIP24 -> mylib2:AD8403-DIP28
- JP2: value PWR -> (none)
- JP4: value LP -> LPFOUT
- JP5: value BP -> BPFOUT
- JP6: value HP -> HPFOUT
- R5: device pot:TRIM_EU-B25P -> rcl:R-EU_0207/7
Connections:
- removed net N$11: C10.2, R1.1, R4.2
- removed net N$15: LED1.C, R7.2
- new net +2V5: JP2.2
- net +5V: no longer LED1.A
- net GND: no longer JP3.2, R5.A, R8.1
- net N$1: now also C10.1, R5.2; no longer R5.E
- net N$12: now also IC1.B4; no longer IC1.B2
- net N$14: now also IC1.A4, IC1.W4, IC2B.+IN, R1.2; no longer LED2.C, R8.2
- net N$2: now also IC1.W2, IC2A.+IN; no longer C10.1, R5.S
- net N$3: now also IC2A.-IN, IC2A.OUT, R1.1; no longer IC1.A2, IC1.W2, IC2A.+IN, R1.2
- net N$4: now also IC2B.-IN; no longer IC2A.-IN
- net N$5: now also IC2B.OUT; no longer IC2A.OUT
- net N$8: now also C10.2, IC1.A2; no longer IC2B.-IN, IC2B.OUT
- net VCC/2: now also IC1.B2, JP3.2, R5.1; no longer IC2B.+IN, JP2.2, JP7.1, JP7.2, LED2.A, R4.1, R7.1
Other:
- moved on the sheet: C10, IC2A, IC2B, JP1, JP2, JP3, R1
