File: eagle/AD8403_SVF/SVF_AC_Coupling.sch (EAGLE design)
At the start: 30 parts, among them IC1 AD8403-DIP24, IC2 NJM2732, IC3 NJM2732

Commit message: Update: eagle files
Parts:
- removed C7: 0.1uF, rcl:C-EU025-024X044
- removed IC1: AD8403-DIP24, mylib2:AD8403-DIP24
- removed JP1: SPI, pinhead:PINHD-1X4
- removed JP7: VGND, pinhead:PINHD-1X2
- removed LED1, LED2: red, led:LED3MM
- C1, C2: device rcl:C-EU050-025X075 -> rcl:C-EU025-025X050
- JP2: value PWR -> (none)
- JP4: value LP -> LPFOUT
- JP5: value BP -> BPFOUT
- JP6: value HP -> HPFOUT
- R6: value 2.2k -> 20k
- R7, R8: value 220 -> 15k
Connections:
- removed net !CS: IC1.!CS, JP1.1
- removed net MOSI: IC1.SDI, JP1.2
- removed net N$12: IC1.B2, R6.1
- removed net N$14: LED2.C, R8.2
- removed net N$15: LED1.C, R7.2
- removed net N$6: C2.1, IC1.A3, IC1.W3, IC3B.-IN
- removed net SCK: IC1.CLK, JP1.3
- new net +2V5: JP2.2
- new net N$13: C2.1, IC3A.-IN, R8.2
- net +5V: no longer C7.1, IC1.!SHDN, IC1.VDD, LED1.A
- net GND: no longer C7.2, IC1.!RS, IC1.AGND1, IC1.AGND2, IC1.AGND3, IC1.AGND4, IC1.DGND, JP1.4, JP3.2, R5.A, R8.1
- net N$10: now also IC2B.OUT, R8.1; no longer IC1.B3, IC3A.OUT
- net N$3: now also R6.1; no longer IC1.A2, IC1.W2
- net N$5: now also R7.1; no longer IC1.B1
- net N$7: now also IC2B.-IN, R7.2; no longer IC1.A1, IC1.W1, IC3A.-IN
- net N$8: now also IC3B.-IN, IC3B.OUT; no longer IC2B.-IN, IC2B.OUT
- net N$9: now also IC3A.OUT; no longer IC3B.OUT
- net VCC/2: now also JP3.2, R5.A; no longer JP2.2, JP7.1, JP7.2, LED2.A, R7.1
Other:
- note removed: "ピンソケットで実装"
- moved on the sheet: IC2B, IC3A, IC3B, R6, R7, R8
